Commit message: fixed URDF and small changes to main file

File: go2_description/urdf/go2_description.urdf (robot description, URDF)
Before this commit: robot go2_description, 41 links, 40 joints
Links:
- link Head_lower: geometry 
- link Head_upper: geometry 
Joints:
- joint FL_calf_joint: limit lower=-2.7227 upper=-0.83776 effort=45.43 velocity=15.70 -> lower=-2.7227 upper=0.3 effort=45.43 velocity=15.70
- joint FR_calf_joint: limit lower=-2.7227 upper=-0.83776 effort=45.43 velocity=15.70 -> lower=-2.7227 upper=0.3 effort=45.43 velocity=15.70
- joint RL_calf_joint: limit lower=-2.7227 upper=-0.83776 effort=45.43 velocity=15.70 -> lower=-2.7227 upper=0.3 effort=45.43 velocity=15.70
- joint RR_calf_joint: limit lower=-2.7227 upper=-0.83776 effort=45.43 velocity=15.70 -> lower=-2.7227 upper=0.3 effort=45.43 velocity=15.70
